Commit message: URDF & ROS2 direction big edit

File: src/macrobot_description/urdf/assemblies/macrobot_full_exact_gripper.urdf.xacro (robot description, xacro)
@@ -399,5 +399,7 @@
       <child link="${prefix}ratio_left_gear"/>
       <origin xyz="0.020950 0.057900 0.064595" rpy="0.000000 -0.000000 -0.000000"/>
-      <axis xyz="0.000000 1.000000 -0.000000"/>
+      <!-- Positive logical q1 is forward tilt. The driven gear rotates opposite
+           the left servo, so its semantic positive axis is -Y. -->
+      <axis xyz="0.000000 -1.000000 0.000000"/>
       <limit effort="100.0" velocity="1.00"/>
     </joint>

File: src/macrobot_description/urdf/assemblies/macrobot_full_visual.urdf.xacro (robot description, xacro)
@@ -399,5 +399,7 @@
       <child link="${prefix}ratio_left_gear"/>
       <origin xyz="0.020950 0.057900 0.064595" rpy="0.000000 -0.000000 -0.000000"/>
-      <axis xyz="0.000000 1.000000 -0.000000"/>
+      <!-- Positive logical q1 is forward tilt. The driven gear rotates opposite
+           the left servo, so its semantic positive axis is -Y. -->
+      <axis xyz="0.000000 -1.000000 0.000000"/>
       <limit effort="100.0" velocity="1.00"/>
     </joint>

File: src/macrobot_description/urdf/macrobot_arm_kinematic.urdf.xacro (robot description, xacro)
@@ -3,7 +3,8 @@
   <!--
     Reduced logical model of the geared four-bar arm and gripper.
-    q1 = arm_lift_joint
-    q2 = wrist_pitch_joint, relative to the main arm
-    q3 = gripper_joint, 0 rad is fully open and negative closes
+    q1 = arm_lift_joint (legacy name): left-servo arm tilt; positive tilts forward
+    q2 = wrist_pitch_joint (legacy name): relative rear-lift coordinate
+         right driven/rear-lift angle = q1 + q2
+    q3 = gripper_joint: 0 rad open; positive closes; pi/2 is full close
     The exact closed mechanisms are visualized by macrobot_full_visual.  This
     model is deliberately simple so FK/IK and joint-limit testing remain robust.
@@ -60,5 +61,5 @@
     <child link="main_arm_link"/>
     <origin xyz="${pivot_x} ${pivot_y} ${pivot_z}" rpy="0 0 0"/>
-    <axis xyz="0 1 0"/>
+    <axis xyz="0 -1 0"/>
     <limit lower="-1.0" upper="1.0" effort="10.0" velocity="1.0"/>
   </joint>
@@ -78,5 +79,5 @@
     <child link="wrist_link"/>
     <origin xyz="0 0 ${main_length}" rpy="0 0 0"/>
-    <axis xyz="0 1 0"/>
+    <axis xyz="0 -1 0"/>
     <limit lower="-1.30" upper="1.30" effort="10.0" velocity="1.0"/>
   </joint>
@@ -98,6 +99,6 @@
     <child link="left_finger_link"/>
     <origin xyz="-0.17215 -0.00390 0.00400" rpy="0 0 1.570796"/>
-    <axis xyz="0 0 1"/>
-    <limit lower="-1.25" upper="0.0" effort="5.0" velocity="1.0"/>
+    <axis xyz="0 0 -1"/>
+    <limit lower="0.0" upper="1.57079632679" effort="5.0" velocity="1.0"/>
   </joint>
   <link name="right_finger_link">
@@ -116,6 +117,6 @@
     <child link="right_finger_link"/>
     <origin xyz="-0.17215 0.00610 0.00400" rpy="0 0 1.570796"/>
-    <axis xyz="0 0 1"/>
-    <limit lower="0.0" upper="1.25" effort="5.0" velocity="1.0"/>
+    <axis xyz="0 0 -1"/>
+    <limit lower="-1.57079632679" upper="0.0" effort="5.0" velocity="1.0"/>
     <mimic joint="gripper_joint" multiplier="-1.0" offset="0.0"/>
   </joint>

Commit message: URDF huge fix

File: src/macrobot_description/urdf/assemblies/macrobot_full_exact_gripper.urdf.xacro (robot description, xacro)
@@ -2,5 +2,5 @@
 <robot xmlns:xacro="http://www.ros.org/wiki/xacro" name="macrobot_exact_gripper_macro">
   <xacro:macro name="macrobot_full_exact_gripper" params="prefix">
-    <!-- Reviewed Fusion export: ros2_control removed, camera TF corrected, nested gripper origins made parent-relative. -->
+    <!-- Corrected Fusion collision export: detailed DAE collisions, physical axis conventions, parent-relative gripper joints, and no generated ros2_control block. -->
     <!-- Links -->
     <link name="${prefix}base_link">
@@ -20,5 +20,5 @@
         <origin xyz="0.000000 0.000000 0.000000" rpy="0 0 0"/>
         <geometry>
-          <mesh filename="package://macrobot_description/meshes/macrobot/base_link_collision.stl" scale="0.01 0.01 0.01"/>
+          <mesh filename="package://macrobot_description/meshes/macrobot/base_link.dae" scale="1 1 1"/>
         </geometry>
       </collision>
@@ -40,5 +40,5 @@
         <origin xyz="-0.020950 -0.041100 -0.039000" rpy="0 0 0"/>
         <geometry>
-          <mesh filename="package://macrobot_description/meshes/macrobot/servo_left_gear_collision.stl" scale="0.01 0.01 0.01"/>
+          <mesh filename="package://macrobot_description/meshes/macrobot/servo_left_gear.dae" scale="1 1 1"/>
         </geometry>
       </collision>
@@ -60,5 +60,5 @@
         <origin xyz="-0.020950 -0.088900 -0.039000" rpy="0 0 0"/>
         <geometry>
-          <mesh filename="package://macrobot_description/meshes/macrobot/servo_right_gear_collision.stl" scale="0.01 0.01 0.01"/>
+          <mesh filename="package://macrobot_description/meshes/macrobot/servo_right_gear.dae" scale="1 1 1"/>
         </geometry>
       </collision>
@@ -80,5 +80,5 @@
         <origin xyz="-0.020950 -0.057900 -0.064595" rpy="0 0 0"/>
         <geometry>
-          <mesh filename="package://macrobot_description/meshes/macrobot/ratio_left_gear_collision.stl" scale="0.01 0.01 0.01"/>
+          <mesh filename="package://macrobot_description/meshes/macrobot/ratio_left_gear.dae" scale="1 1 1"/>
         </geometry>
       </collision>
@@ -100,5 +100,5 @@
         <origin xyz="-0.020950 -0.072300 -0.064595" rpy="0 0 0"/>
         <geometry>
-          <mesh filename="package://macrobot_description/meshes/macrobot/ratio_right_gear_collision.stl" scale="0.01 0.01 0.01"/>
+          <mesh filename="package://macrobot_description/meshes/macrobot/ratio_right_gear.dae" scale="1 1 1"/>
         </geometry>
       </collision>
@@ -120,5 +120,5 @@
         <origin xyz="-0.037000 -0.148700 -0.019300" rpy="0 0 0"/>
         <geometry>
-          <mesh filename="package://macrobot_description/meshes/macrobot/front_right_wheel_collision.stl" scale="0.01 0.01 0.01"/>
+          <mesh filename="package://macrobot_description/meshes/macrobot/front_right_wheel.dae" scale="1 1 1"/>
         </geometry>
       </collision>
@@ -140,5 +140,5 @@
         <origin xyz="-0.123500 -0.148700 -0.019300" rpy="0 0 0"/>
         <geometry>
-          <mesh filename="package://macrobot_description/meshes/macrobot/back_right_wheel_collision.stl" scale="0.01 0.01 0.01"/>
+          <mesh filename="package://macrobot_description/meshes/macrobot/back_right_wheel.dae" scale="1 1 1"/>
         </geometry>
       </collision>
@@ -160,5 +160,5 @@
         <origin xyz="-0.037000 0.018700 -0.019300" rpy="0 0 0"/>
         <geometry>
-          <mesh filename="package://macrobot_description/meshes/macrobot/front_left_wheel_collision.stl" scale="0.01 0.01 0.01"/>
+          <mesh filename="package://macrobot_description/meshes/macrobot/front_left_wheel.dae" scale="1 1 1"/>
         </geometry>
       </collision>
@@ -180,9 +180,12 @@
         <origin xyz="-0.123500 0.018700 -0.019300" rpy="0 0 0"/>
         <geometry>
-          <mesh filename="package://macrobot_description/meshes/macrobot/back_left_wheel_collision.stl" scale="0.01 0.01 0.01"/>
+          <mesh filename="package://macrobot_description/meshes/macrobot/back_left_wheel.dae" scale="1 1 1"/>
         </geometry>
       </collision>
     </link>
     <link name="${prefix}camera_link">
+      <!-- camera_link is the D435F depth reference point.  The exported marker
+           mesh is base-relative, so its local origin is shifted by the negative
+           base_link -> camera_link translation. -->
       <inertial>
         <origin xyz="0 0 0" rpy="0 0 0"/>
@@ -191,7 +194,7 @@
       </inertial>
       <visual>
-        <origin xyz="0 0 0" rpy="0 0 0"/>
-        <geometry>
-          <sphere radius="0.0035"/>
+        <origin xyz="0.030850 0.000413 -0.017858" rpy="0 0 0"/>
+        <geometry>
+          <mesh filename="package://macrobot_description/meshes/macrobot/camera_link.dae" scale="1 1 1"/>
         </geometry>
         <material name="camera_marker">
@@ -199,4 +202,10 @@
         </material>
       </visual>
+      <collision>
+        <origin xyz="0.030850 0.000413 -0.017858" rpy="0 0 0"/>
+        <geometry>
+          <mesh filename="package://macrobot_description/meshes/macrobot/camera_link.dae" scale="1 1 1"/>
+        </geometry>
+      </collision>
     </link>
     <link name="${prefix}back_link">
@@ -216,5 +225,5 @@
         <origin xyz="-0.048950 -0.076600 -0.064595" rpy="0 0 0"/>
         <geometry>
-          <mesh filename="package://macrobot_description/meshes/macrobot/back_link_collision.stl" scale="0.01 0.01 0.01"/>
+          <mesh filename="package://macrobot_description/meshes/macrobot/back_link.dae" scale="1 1 1"/>
         </geometry>
       </collision>

File: src/macrobot_description/urdf/assemblies/macrobot_full_visual.urdf.xacro (robot description, xacro)
@@ -2,5 +2,5 @@
 <robot xmlns:xacro="http://www.ros.org/wiki/xacro" name="macrobot_macro">
   <xacro:macro name="macrobot_full_visual" params="prefix">
-    <!-- Reviewed Fusion export: ros2_control removed, camera TF corrected, nested gripper origins made parent-relative. -->
+    <!-- Corrected Fusion collision export: detailed DAE collisions, physical axis conventions, parent-relative gripper joints, and no generated ros2_control block. -->
     <!-- Links -->
     <link name="${prefix}base_link">
@@ -20,5 +20,5 @@
         <origin xyz="0.000000 0.000000 0.000000" rpy="0 0 0"/>
         <geometry>
-          <mesh filename="package://macrobot_description/meshes/macrobot/base_link_collision.stl" scale="0.01 0.01 0.01"/>
+          <mesh filename="package://macrobot_description/meshes/macrobot/base_link.dae" scale="1 1 1"/>
         </geometry>
       </collision>
@@ -40,5 +40,5 @@
         <origin xyz="-0.020950 -0.041100 -0.039000" rpy="0 0 0"/>
         <geometry>
-          <mesh filename="package://macrobot_description/meshes/macrobot/servo_left_gear_collision.stl" scale="0.01 0.01 0.01"/>
+          <mesh filename="package://macrobot_description/meshes/macrobot/servo_left_gear.dae" scale="1 1 1"/>
         </geometry>
       </collision>
@@ -60,5 +60,5 @@
         <origin xyz="-0.020950 -0.088900 -0.039000" rpy="0 0 0"/>
         <geometry>
-          <mesh filename="package://macrobot_description/meshes/macrobot/servo_right_gear_collision.stl" scale="0.01 0.01 0.01"/>
+          <mesh filename="package://macrobot_description/meshes/macrobot/servo_right_gear.dae" scale="1 1 1"/>
         </geometry>
       </collision>
@@ -80,5 +80,5 @@
         <origin xyz="-0.020950 -0.057900 -0.064595" rpy="0 0 0"/>
         <geometry>
-          <mesh filename="package://macrobot_description/meshes/macrobot/ratio_left_gear_collision.stl" scale="0.01 0.01 0.01"/>
+          <mesh filename="package://macrobot_description/meshes/macrobot/ratio_left_gear.dae" scale="1 1 1"/>
         </geometry>
       </collision>
@@ -100,5 +100,5 @@
         <origin xyz="-0.020950 -0.072300 -0.064595" rpy="0 0 0"/>
         <geometry>
-          <mesh filename="package://macrobot_description/meshes/macrobot/ratio_right_gear_collision.stl" scale="0.01 0.01 0.01"/>
+          <mesh filename="package://macrobot_description/meshes/macrobot/ratio_right_gear.dae" scale="1 1 1"/>
         </geometry>
       </collision>
@@ -120,5 +120,5 @@
         <origin xyz="-0.037000 -0.148700 -0.019300" rpy="0 0 0"/>
         <geometry>
-          <mesh filename="package://macrobot_description/meshes/macrobot/front_right_wheel_collision.stl" scale="0.01 0.01 0.01"/>
+          <mesh filename="package://macrobot_description/meshes/macrobot/front_right_wheel.dae" scale="1 1 1"/>
         </geometry>
       </collision>
@@ -140,5 +140,5 @@
         <origin xyz="-0.123500 -0.148700 -0.019300" rpy="0 0 0"/>
         <geometry>
-          <mesh filename="package://macrobot_description/meshes/macrobot/back_right_wheel_collision.stl" scale="0.01 0.01 0.01"/>
+          <mesh filename="package://macrobot_description/meshes/macrobot/back_right_wheel.dae" scale="1 1 1"/>
         </geometry>
       </collision>
@@ -160,5 +160,5 @@
         <origin xyz="-0.037000 0.018700 -0.019300" rpy="0 0 0"/>
         <geometry>
-          <mesh filename="package://macrobot_description/meshes/macrobot/front_left_wheel_collision.stl" scale="0.01 0.01 0.01"/>
+          <mesh filename="package://macrobot_description/meshes/macrobot/front_left_wheel.dae" scale="1 1 1"/>
         </geometry>
       </collision>
@@ -180,9 +180,12 @@
         <origin xyz="-0.123500 0.018700 -0.019300" rpy="0 0 0"/>
         <geometry>
-          <mesh filename="package://macrobot_description/meshes/macrobot/back_left_wheel_collision.stl" scale="0.01 0.01 0.01"/>
+          <mesh filename="package://macrobot_description/meshes/macrobot/back_left_wheel.dae" scale="1 1 1"/>
         </geometry>
       </collision>
     </link>
     <link name="${prefix}camera_link">
+      <!-- camera_link is the D435F depth reference point.  The exported marker
+           mesh is base-relative, so its local origin is shifted by the negative
+           base_link -> camera_link translation. -->
       <inertial>
         <origin xyz="0 0 0" rpy="0 0 0"/>
@@ -191,7 +194,7 @@
       </inertial>
       <visual>
-        <origin xyz="0 0 0" rpy="0 0 0"/>
-        <geometry>
-          <sphere radius="0.0035"/>
+        <origin xyz="0.030850 0.000413 -0.017858" rpy="0 0 0"/>
+        <geometry>
+          <mesh filename="package://macrobot_description/meshes/macrobot/camera_link.dae" scale="1 1 1"/>
         </geometry>
         <material name="camera_marker">
@@ -199,4 +202,10 @@
         </material>
       </visual>
+      <collision>
+        <origin xyz="0.030850 0.000413 -0.017858" rpy="0 0 0"/>
+        <geometry>
+          <mesh filename="package://macrobot_description/meshes/macrobot/camera_link.dae" scale="1 1 1"/>
+        </geometry>
+      </collision>
     </link>
     <link name="${prefix}back_link">
@@ -216,5 +225,5 @@
         <origin xyz="-0.048950 -0.076600 -0.064595" rpy="0 0 0"/>
         <geometry>
-          <mesh filename="package://macrobot_description/meshes/macrobot/back_link_collision.stl" scale="0.01 0.01 0.01"/>
+          <mesh filename="package://macrobot_description/meshes/macrobot/back_link.dae" scale="1 1 1"/>
         </geometry>
       </collision>
@@ -236,5 +245,5 @@
         <origin xyz="-0.048950 -0.073200 -0.164595" rpy="0 0 0"/>
         <geometry>
-          <mesh filename="package://macrobot_description/meshes/macrobot/gripper_link_collision.stl" scale="0.01 0.01 0.01"/>
+          <mesh filename="package://macrobot_description/meshes/macrobot/gripper_link.dae" scale="1 1 1"/>
         </geometry>
       </collision>
@@ -256,5 +265,5 @@
         <origin xyz="-0.217623 -0.105919 -0.108635" rpy="0 0 0"/>
         <geometry>
-          <mesh filename="package://macrobot_description/meshes/macrobot/gripper_servo_gear_collision.stl" scale="0.01 0.01 0.01"/>
+          <mesh filename="package://macrobot_description/meshes/macrobot/gripper_servo_gear.dae" scale="1 1 1"/>
         </geometry>
       </collision>
@@ -276,5 +285,5 @@
         <origin xyz="-0.211064 -0.122690 -0.169095" rpy="0 0 0"/>
         <geometry>
-          <mesh filename="package://macrobot_description/meshes/macrobot/gripper_left_gear_collision.stl" scale="0.01 0.01 0.01"/>
+          <mesh filename="package://macrobot_description/meshes/macrobot/gripper_left_gear.dae" scale="1 1 1"/>
         </geometry>
       </collision>
@@ -296,5 +305,5 @@
         <origin xyz="-0.235064 -0.122690 -0.169095" rpy="0 0 0"/>
         <geometry>
-          <mesh filename="package://macrobot_description/meshes/macrobot/gripper_right_gear_collision.stl" scale="0.01 0.01 0.01"/>
+          <mesh filename="package://macrobot_description/meshes/macrobot/gripper_right_gear.dae" scale="1 1 1"/>
         </geometry>
       </collision>
@@ -316,5 +325,5 @@
         <origin xyz="-0.218064 -0.137690 -0.169095" rpy="0 0 0"/>
         <geometry>
-          <mesh filename="package://macrobot_description/meshes/macrobot/gripper_left_addition_collision.stl" scale="0.01 0.01 0.01"/>
+          <mesh filename="package://macrobot_description/meshes/macrobot/gripper_left_addition.dae" scale="1 1 1"/>
         </geometry>
       </collision>
@@ -336,5 +345,5 @@
         <origin xyz="-0.228064 -0.137690 -0.169095" rpy="0 0 0"/>
         <geometry>
-          <mesh filename="package://macrobot_description/meshes/macrobot/gripper_right_addition_collision.stl" scale="0.01 0.01 0.01"/>
+          <mesh filename="package://macrobot_description/meshes/macrobot/gripper_right_addition.dae" scale="1 1 1"/>
         </geometry>
       </collision>
@@ -356,5 +365,5 @@
         <origin xyz="-0.188064 -0.137690 -0.168595" rpy="0 0 0"/>
         <geometry>
-          <mesh filename="package://macrobot_description/meshes/macrobot/gripper_clamp_left_collision.stl" scale="0.01 0.01 0.01"/>
+          <mesh filename="package://macrobot_description/meshes/macrobot/gripper_clamp_left.dae" scale="1 1 1"/>
         </geometry>
       </collision>
@@ -376,5 +385,5 @@
         <origin xyz="-0.258064 -0.137690 -0.168595" rpy="0 0 0"/>
         <geometry>
-          <mesh filename="package://macrobot_description/meshes/macrobot/gripper_clamp_right_collision.stl" scale="0.01 0.01 0.01"/>
+          <mesh filename="package://macrobot_description/meshes/macrobot/gripper_clamp_right.dae" scale="1 1 1"/>
         </geometry>
       </collision>

File: src/macrobot_description/urdf/macrobot_arm_kinematic.urdf.xacro (robot description, xacro)
@@ -30,5 +30,5 @@
       <origin xyz="0 0 0" rpy="0 0 0"/>
       <geometry>
-        <mesh filename="package://macrobot_description/meshes/macrobot/base_link_collision.stl" scale="0.01 0.01 0.01"/>
+        <mesh filename="package://macrobot_description/meshes/macrobot/base_link.dae" scale="1 1 1"/>
       </geometry>
     </collision>

File: src/macrobot_description/urdf/macrobot_full_collision.urdf.xacro (robot description, xacro)
@@ -1,5 +1,5 @@
 <?xml version="1.0"?>
 <robot xmlns:xacro="http://www.ros.org/wiki/xacro" name="macrobot_full_collision">
-  <!-- Full Fusion link tree with the exported per-link collision geometry. -->
+  <!-- Full Fusion link tree with the corrected detailed DAE collision geometry. -->
   <material name="material"><color rgba="0.965 0.965 0.953 1.0"/></material>
   <xacro:include filename="$(find macrobot_description)/urdf/assemblies/macrobot_full_visual.urdf.xacro"/>

File: src/macrobot_description/urdf/macrobot_full_exact_gripper.urdf.xacro (robot description, xacro)
@@ -1,5 +1,5 @@
 <?xml version="1.0"?>
 <robot xmlns:xacro="http://www.ros.org/wiki/xacro" name="macrobot_full_exact_gripper">
-  <!-- Full Fusion tree; detailed visual meshes are reused for gripper collision. -->
+  <!-- Full reviewed Fusion tree; corrected detailed DAE collision geometry is used for every physical link. -->
   <material name="material"><color rgba="0.965 0.965 0.953 1.0"/></material>
   <xacro:include filename="$(find macrobot_description)/urdf/assemblies/macrobot_full_exact_gripper.urdf.xacro"/>
